File: hw/sch_pcb/_autosave-AMFOC01.kicad_pcb (KiCad board)
At the start: 2 copper layers, 70.9 x 60.8 mm, 102 parts, among them J1 USBC_USB4105-GF-A, J10 OLED, J11 Jack-DC, J12 Mini-DIN-4, J2 Conn_01x01, J3 Conn_01x01, J4 Conn_01x01, J5 Conn_01x02, J6 Conn_01x04, J7 Conn_01x04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

Commit message: oprava chyb
Parts:
- R22, R23: value 10k -> 0R15
- moved R29 2.10 mm to (113.8, 113.0), turned to 180 degrees
Connections:
- J10 pad 10: unconnected-(J10-Pad10) -> GND
- J10 pad 11: unconnected-(J10-Pad11) -> GND
- J10 pad 12: unconnected-(J10-Pad12) -> GND
- R29 pad 1: +3V3 -> Net-(J10-Pad26)
- R29 pad 2: Net-(J10-Pad26) -> GND
Routing:
- net +3V3: track 245.2 -> 239.6 mm, vias 15 -> 14
- net Net-(J10-Pad26): track 10.8 -> 8.20 mm
- net GND: vias 61 -> 60
